File: PCB/TinyNumberHat.kicad_pcb (KiCad board)
At the start: 4 copper layers, 65 x 30 mm, 38 parts, among them IC1 SamacSys_Parts_HT16K33-28SOP, J1 GPIO, J2 SM04B-SRSS-TB(LF)(SN), SW1 SW_Omron_B3FS, SW2 SW_Omron_B3FS, SW3 SW_Omron_B3FS, SW4 SW_Omron_B3FS

Commit message: Update to Kicad 9, add schematic
Other:
- board text added: "3.3v"
- board text added: "5v"
- board text added: "By ADRE"
- board text added: "TinyNumberHat"
- board text added: "ver 1.0"
- board text removed: "locked"
