File: PCB/TinyNumberHat.kicad_sch (KiCad schematic)
At the start: 32 parts, among them IC1 SamacSys_Parts_HT16K33-28SOP, J1 GPIO, J3 SM04B-SRSS-TB(LF)(SN), SW1 SW_Omron_B3FS, SW2 SW_Omron_B3FS, SW3 SW_Omron_B3FS, SW4 SW_Omron_B3FS

Commit message: WIP
Parts:
- removed C11 (x2): 10uF, Capacitor_SMD:C_0603_1608Metric, symbol Device:C_Small
- removed C7: 15uF, Capacitor_SMD:C_1210_3225Metric_Pad1.33x2.70mm_HandSolder, symbol Device:C_Small
- removed J3: SM04B-SRSS-TB(LF)(SN), LTP-305G:JST_SM04B-SRSS-TB(LF)(SN), symbol SM04B-SRSS-TB_LF__SN_:SM04B-SRSS-TB(LF)(SN)
- removed R3: 47k, Resistor_SMD:R_0603_1608Metric, symbol Device:R
- removed R3: 10k, Resistor_SMD:R_0603_1608Metric, symbol Device:R
- added C1: 15uF, Capacitor_SMD:C_1210_3225Metric_Pad1.33x2.70mm_HandSolder, symbol Device:C_Small
- added C3, C4: 10uF, Capacitor_SMD:C_0603_1608Metric, symbol Device:C_Small
- added J2: SM04B-SRSS-TB(LF)(SN), LTP-305G:JST_SM04B-SRSS-TB(LF)(SN), symbol SM04B-SRSS-TB_LF__SN_:SM04B-SRSS-TB(LF)(SN)
- added R6: 47k, Resistor_SMD:R_0603_1608Metric, symbol Device:R
- added R7: 10k, Resistor_SMD:R_0603_1608Metric, symbol Device:R
Connections:
- net GND: now also C1.1, C3.2, C4.2, J2.1, J2.S1 (SHIELD), J2.S2 (SHIELD)
- net GPIO2/SDA1: now also J2.3, R6.1
- net GPIO3/SCL1: now also J2.4, R7.1
- net power: now also C1.2, C3.1, C4.1, J2.2, R6.2, R7.2

Commit message: Update to Kicad 9, add schematic
Parts:
- renumbered C11 to C2, D3 to D1, D3 to D2, R3 to R1, R3 to R2, R3 to R4, R3 to R5, R3 to R8, R3 to R9
